Commit message: control in gazebo *commands* colcon build --symlink-install source install/setup.bash ros2 launch humble_bot launch_sim.launch.py ros2 run teleop_twist_keyboard teleop_twist_keyboard *save frame ** ros2 run tf2_tools view_frames

File: description/robot_core.xacro (robot description, xacro)
@@ -1,6 +1,5 @@
 <?xml version="1.0"?>
 <robot xmlns:xacro="http://www.ros.org/wiki/xacro" >
-    <xacro:include filename="inertial_macros.xacro" />
-    <!-- MATERIALS -->
+    <xacro:include filename="inertial_macros.xacro"/>
     <material name="white">
         <color rgba="1 1 1 1" />
@@ -45,5 +44,5 @@
         <material>Gazebo/White</material>
     </gazebo>
-        <!-- LEFT WHEEL LINK -->
+    <!-- LEFT WHEEL LINK -->
     <joint name="left_wheel_joint" type="continuous">
         <parent link="base_link"/>
@@ -108,5 +107,5 @@
                 <sphere radius="0.05"/>
             </geometry>
-            <material name="black"/>
+            <material name="orange"/>
         </visual>
         <collision>
@@ -120,7 +119,7 @@
     </link>
     <gazebo reference="caster_wheel">
-        <material>Gazebo/Black</material>
-        <mu1 value="0.001" />
-        <mu2 value="0.001" />
+        <material>Gazebo/Orange</material>
+        <mu1 value="0.001"/>  <!-- Трение в направлении движения -->
+        <mu2 value="0.001"/> <!-- Трение в боковом направлении -->
     </gazebo>
 </robot>
